Commit message: Update hokuyo.urdf.xacro

File: hokuyo.urdf.xacro (robot description, xacro)
@@ -5,10 +5,10 @@
   <!-- Hokuyo 2D LIDAR -->
   <xacro:macro name="sensor_hokuyo" params="parent">
-		<joint name="laser" type="fixed">
+    <joint name="laser" type="fixed">
       <origin xyz="0.1 0.0 0.43" rpy="0 0 0" />
       <parent link="base_link" />
       <child link="base_laser_link" />
     </joint>
-		<link name="base_laser_link">
+<link name="base_laser_link">
       <visual>
         <geometry>
@@ -17,14 +17,14 @@
       </visual>
       <collision>
-				<origin xyz="0 0 -0.0145" rpy="0 0 0" />
-					<geometry>
-						<box size="0.05 0.05 0.041"/>
-					</geometry>
+	<origin xyz="0 0 -0.0145" rpy="0 0 0" />
+	<geometry>
+	  <box size="0.05 0.05 0.041"/>
+	</geometry>
       </collision>
       <collision>
-				<origin xyz="0 0 0.0205" rpy="0 0 0" />
-					<geometry>
-						<cylinder radius="0.021" length="0.029"/>
-					</geometry>
+	<origin xyz="0 0 0.0205" rpy="0 0 0" />
+	<geometry>
+	  <cylinder radius="0.021" length="0.029"/>
+	</geometry>
       </collision>
       <inertial>
@@ -32,6 +32,6 @@
         <origin xyz="0 0 0" />
         <inertia ixx="0.0001" ixy="0.0" ixz="0.0" iyy="0.0001" iyz="0.0" izz="0.0001" />
-			</inertial>
-		</link>
+      </inertial>
+</link>
 	<!-- Hokuyo sensor for simulation -->
     <hokuyo_laser />
